Commit message: add ycb

File: examples/ycb/006_mustard_bottle.urdf (robot description, URDF)
Before this commit: robot 006_mustard_bottle, 1 links, 0 joints
Links:
- link _name: geometry collision mesh filename=006_mustard_bottle/google_16k/textured_vhacd.obj scale=1 1 1; visual mesh filename=006_mustard_bottle/google_16k/textured.obj scale=1 1 1

File: examples/ycb/_prototype.urdf (robot description, URDF)
Before this commit: robot _name, 1 links, 0 joints
Links:
- link _name: geometry collision mesh filename=_prototype.obj scale=1 1 1; visual mesh filename=_prototype.obj scale=1 1 1
